File: BoostBoard/BoastBoard.sch (KiCad schematic (older format))
At the start: 15 parts

Commit message: Made more work on the boostboard>
Parts:
- removed C?: C, symbol C
- removed D?: D, symbol D
- removed P?: CONN_01X02, symbol CONN_01X02
- added P1: USB_B, Connect:USB_B, symbol USB_B
- added P3: CONN_01X03, Pin_Headers:Pin_Header_Straight_1x03, symbol CONN_01X03
- added R1_2: 18k, Resistors_ThroughHole:Resistor_Vertical_RM5mm, symbol R
- C_T1: renamed from C?; value C_T -> 330uF; footprint (none) -> Capacitors_ThroughHole:C_Radial_D10_L13_P5
- Co1: renamed from Co; value 330uF -> 47uF; footprint (none) -> Capacitors_ThroughHole:C_Radial_D10_L13_P5
- D2: renamed from D?; footprint (none) -> LEDs:LED-5MM
- D3: renamed from D?; footprint (none) -> Diodes_ThroughHole:Diode_P600_Vertical_AnodeUp
- L1: renamed from L?; value 170uH -> 18uH; footprint (none) -> Choke_Toroid_ThroughHole:Choke_Toroid_horizontal_Diameter12-5mm_Amidon-T44
- P2: renamed from P?; footprint (none) -> Connectors_Molex:Molex_KK-6410-02_02x2.54mm_Straight
- R1, R2: renamed from R?; footprint (none) -> Resistors_ThroughHole:Resistor_Vertical_RM5mm
- R1_1: renamed from R1_; value R -> 36k; footprint (none) -> Resistors_ThroughHole:Resistor_Vertical_RM5mm
- R2_1: renamed from R2_; footprint (none) -> Resistors_ThroughHole:Resistor_Vertical_RM5mm
- REG1: footprint (none) -> Power_Integrations:PDIP-8
- Rsc1: renamed from Rsc; value 0R22 -> 0R15; footprint (none) -> Resistors_ThroughHole:Resistor_Vertical_RM5mm
Connections:
- net GND: now also P1.4 (GND), P1.5 (shield), R1_2.2
- net INV_IN: now also P3.2 (P2); no longer R1_1.1
- net VCC: now also P1.1 (VCC)
- new net: P3.1 (P1), R1_1.1
- new net: P3.3 (P3), R1_2.1
- no-connect marks 0 -> 2
Other:
- moved on the sheet: R1_1
